Commit message: update bumperbot urdf with collision and inertial

File: bumperbot_ws/install/bumperbot_description/share/bumperbot_description/urdf/bumperbot.urdf.xacro (robot description, xacro)
@@ -4,4 +4,11 @@
     <link name="base_footprint"/>
     <link name="base_link">
+        <inertial>
+            <origin xyz="0 0 0.04" rpy="0.0 0.25 0.3" />
+            <mass value="8.2573504e-01"/>
+            <inertia ixx="2.2124416e-02" ixy="-1.2294101e-04" ixz="3.4938785e-04"
+                     iyy="2.1193702e-02" iyz="-5.0120904e-05"
+                     izz="2.0064271e-02" />
+        </inertial>
         <visual>
             <origin rpy="0 0 0" xyz="0 0 0"/>
@@ -10,4 +17,10 @@
             </geometry>
         </visual>
+        <collision>
+            <origin xyz="0 0 0" rpy="0 0 0" />
+            <geometry>
+                <mesh filename="package://bumperbot_description/meshes/base_link.STL" />
+            </geometry>
+        </collision>
     </link>
     <joint name="base_joint" type="fixed">
@@ -17,4 +30,11 @@
     </joint>
     <link name="wheel_right_link">
+        <inertial>
+            <origin xyz="0 -0.014 0" rpy="0 0 0" />
+            <mass value="0.0530086090966721" />
+           <inertia ixx="1.88176298336665E-05" ixy="-4.8444933029987E-10" ixz="1.88163708851143E-08"
+                    iyy="3.11510738647764E-05" iyz="-6.93560663069607E-11"
+                    izz="1.8801969558182E-05" />
+        </inertial>
         <visual>
             <origin rpy="1.57 0 0" xyz="0 0 0"/>
@@ -23,4 +43,10 @@
             </geometry>
         </visual>
+        <collision>
+            <origin xyz="0 -0.015 0" rpy="1.57 0 0" />
+            <geometry>
+                <sphere radius="0.033"/>
+            </geometry>
+        </collision>
     </link>
     <joint name="wheel_right_joint" type="continuous">
@@ -31,4 +57,11 @@
     </joint>
     <link name="wheel_left_link">
+        <inertial>
+            <origin xyz="0 0.014 0" rpy="0 0 0" />
+            <mass value="0.0530086043217644" />
+            <inertia ixx="1.8792911368909E-05"  ixy="3.31256392204584E-10" ixz="-1.14082001662767E-08"
+                     iyy="3.11510738759073E-05" iyz="-3.60499245082192E-10"
+                     izz="1.88266886146847E-05" />
+        </inertial>
         <visual>
             <origin rpy="-1.57 0 0" xyz="0 0 0"/>
@@ -37,4 +70,10 @@
             </geometry>
         </visual>
+        <collision>
+            <origin xyz="0 0.015 0" rpy="-1.57 0 0" />
+            <geometry>
+                <sphere radius="0.033"/>
+            </geometry>
+        </collision>
     </link>
     <joint name="wheel_left_joint" type="continuous">
@@ -45,4 +84,11 @@
     </joint>
     <link name="caster_rear_link">
+        <inertial>
+            <origin xyz="3.8996812895542E-07 2.40073004698083E-07 0.00219173397061509" rpy="0 0 0" />
+            <mass value="1.44379265037902E-06" />
+            <inertia ixx="7.23075276010246E-11" ixy="-6.10956872363424E-16" ixz="2.22849693527207E-15"
+                     iyy="3.87137930859167E-11" iyz="2.939098587861E-15"
+                     izz="1.00967486676306E-10" />
+        </inertial>
         <visual>
             <origin rpy="0 0 0" xyz="0 0 0"/>
@@ -51,4 +97,10 @@
             </geometry>
         </visual>
+        <collision>
+            <origin xyz="0 0 0" rpy="0 0 0" />
+            <geometry>
+                <sphere radius="0.005"/>
+            </geometry>
+        </collision>
     </link>
     <joint name="caster_rear_joint" type="fixed">
@@ -58,4 +110,11 @@
     </joint>
     <link name="caster_front_link">
+        <inertial>
+            <origin xyz="3.89968128948481E-07 2.40073004698083E-07 0.00219173397061506" rpy="0 0 0" />
+            <mass value="1.44379265037903E-06" />
+            <inertia ixx="7.23075276010246E-11" ixy="-6.10956883467859E-16" ixz="2.22849693525031E-15"
+                     iyy="3.8713793085917E-11"  iyz="2.93909858781952E-15"
+                     izz="1.00967486676306E-10" />
+        </inertial>
         <visual>
             <origin rpy="0 0 0" xyz="0 0 0"/>
@@ -64,4 +123,10 @@
             </geometry>
         </visual>
+        <collision>
+            <origin xyz="0 0 0" rpy="0 0 0" />
+            <geometry>
+                <sphere radius="0.005"/>
+            </geometry>
+        </collision>
     </link>
     <joint name="caster_front_joint" type="fixed">
@@ -70,16 +135,3 @@
         <origin rpy="0 0 0" xyz="0.04755 0 -0.027"/>
     </joint>
-    <link name="can_link">
-        <visual>
-            <origin rpy="0 0 0" xyz="0 0 0" />
-            <geometry>
-                <mesh filename="package://bumperbot_description/meshes/can.STL"/>
-            </geometry>
-        </visual>
-    </link>
-    <joint name="can_joint" type="fixed">
-        <parent link="base_link"/>
-        <child link="can_link"/>
-        <origin rpy="1.57 0 0" xyz="-0.03 0.03 0.078"/>
-    </joint>
 </robot>

Commit message: until 46 th video

File: bumperbot_ws/install/bumperbot_description/share/bumperbot_description/urdf/bumperbot.urdf.xacro (robot description, xacro)
@@ -2,4 +2,6 @@
 <robot xmlns:xacro="http://www.ros.org/wiki/xacro" name="bumperbot">
 <!-- xmlns:xacro=... enables use of Xacro macros (not used in this snippet, but allows future extensions).-->
+    <!-- Include Gazebo Parameters -->
+    <xacro:include filename="$(find bumperbot_description)/urdf/bumperbot_gazebo.xacro"/>
     <link name="base_footprint"/>
     <link name="base_link">
@@ -17,5 +19,5 @@
             </geometry>
         </visual>
-        <collision>
+        <collision>        <!-- The collision block defines how the simulator (Gazebo, Isaac, Webots, etc.) should treat a link when it touches other objects in the environment.-->
             <origin xyz="0 0 0" rpy="0 0 0" />
             <geometry>
@@ -31,5 +33,5 @@
     <link name="wheel_right_link">
         <inertial>
-            <origin xyz="0 -0.014 0" rpy="0 0 0" />
+            <origin xyz="0 -0.014 0" rpy="0 0 0" />  <!-- where the center of mass (CoM) is located in the link’s frame-->
             <mass value="0.0530086090966721" />
            <inertia ixx="1.88176298336665E-05" ixy="-4.8444933029987E-10" ixz="1.88163708851143E-08"
@@ -44,7 +46,7 @@
         </visual>
         <collision>
-            <origin xyz="0 -0.015 0" rpy="1.57 0 0" />
+            <origin xyz="0 -0.015 0" rpy="1.57 0 0" />      <!-- Ensures that the sphere touches the ground at the right place (aligned with the wheel rim). -->
             <geometry>
-                <sphere radius="0.033"/>
+                <sphere radius="0.033"/>       <!-- Sphere collision is computationally the simplest shape. less jitter, faster, smoother rolling.-->
             </geometry>
         </collision>
